File: KiCadFiles/FaultSignalGenerator/FaultSignalGenerator_Isaiah.kicad_pcb (KiCad board)
At the start: 2 copper layers, 0 parts

Commit message: PCB diagram
Working draft on PCB. Started scratching my head on how to get this set up properly. Going to tackle some more over the weekend. Feel free to take a crack if you're game.
Parts:
- added C1: 4700pF, Capacitor_SMD:C_1812_4532Metric_Pad1.57x3.40mm_HandSolder, F.Cu at (74.3, 74.7)
- added C2: 470pF, Capacitor_SMD:C_1812_4532Metric_Pad1.57x3.40mm_HandSolder, F.Cu at (101.6, 61.4)
- added C3: 10u, Capacitor_SMD:C_1812_4532Metric_Pad1.57x3.40mm_HandSolder, F.Cu at (111.8, 61.4)
- added C4: 10uF, Capacitor_SMD:C_1812_4532Metric_Pad1.57x3.40mm_HandSolder, F.Cu at (113.3, 99.1)
- added C5: 100nF, Capacitor_SMD:C_1812_4532Metric_Pad1.57x3.40mm_HandSolder, F.Cu at (88.3, 96.3)
- added C6: 100nF, Capacitor_SMD:C_1812_4532Metric_Pad1.57x3.40mm_HandSolder, F.Cu at (82.5, 96.3)
- added C7: 100nF, Capacitor_SMD:C_1812_4532Metric_Pad1.57x3.40mm_HandSolder, F.Cu at (76.8, 96.3)
- added J1: Conn_02x20_Counter_Clockwise, Connector_JAE:JAE_LY20-40P-DT1_2x20_P2.00mm_Vertical, F.Cu at (161.6, 64.8)
- added R1: 6.2k, Resistor_SMD:R_0603_1608Metric_Pad0.98x0.95mm_HandSolder, F.Cu at (68.6, 77.8)
- added R2: 6.8k, Resistor_SMD:R_0603_1608Metric_Pad0.98x0.95mm_HandSolder, F.Cu at (91.4, 108.2)
- added R3: 430, Resistor_SMD:R_0603_1608Metric_Pad0.98x0.95mm_HandSolder, F.Cu at (94.0, 104.1)
- added R4: 47, Resistor_SMD:R_0603_1608Metric_Pad0.98x0.95mm_HandSolder, F.Cu at (102.2, 104.1)
- added R5: 1k, Resistor_SMD:R_0603_1608Metric_Pad0.98x0.95mm_HandSolder, F.Cu at (108.6, 103.1)
- added R6: 10k, Resistor_SMD:R_0603_1608Metric_Pad0.98x0.95mm_HandSolder, F.Cu at (111.1, 103.1)
- added U1: TL074CDR, TL074CDR_OpAmp:TL074CDR, F.Cu at (101.7, 85.1)
- added U2: MCP4462-502E/ST, DPOT:MCP4462-502E&slash_ST, F.Cu at (114.3, 86.1)
- added U3: PCM1681PWP, PCM1681PWP:PCM1681PWP, F.Cu at (78.7, 86.4)
Routing:
- net 0: track 0.00 -> 155.4 mm
- net Net-(C2-Pad2): track 0.00 -> 130.7 mm
- net Net-(C1-Pad1): track 0.00 -> 79.4 mm
- net +3.3V: track 0.00 -> 47.0 mm
- net +1V5: track 0.00 -> 32.5 mm
- net Net-(R5-Pad1): track 0.00 -> 31.4 mm
- net Net-(C2-Pad1): track 0.00 -> 25.4 mm
- net Net-(C4-Pad1): track 0.00 -> 22.3 mm
- net DAC: track 0.00 -> 9.03 mm
- net Net-(U1-Pad8): track 0.00 -> 8.19 mm
- net out: track 0.00 -> 5.72 mm
- net (no net): track 0.00 -> 2.41 mm
