File: KiCadFiles/FaultSignalGenerator/power.kicad_sch (KiCad schematic)
At the start: 13 parts, among them U16 TL780-05CKTTR

Commit message: Changed 138.1k resistor size
Parts:
- R142: footprint Resistor_SMD:R_1206_3216Metric -> Resistor_SMD:R_0603_1608Metric
Changed lines of the file:
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@@
       (effects (font (size 1.27 1.27)))
     )
-    (property "Footprint" "Resistor_SMD:R_1206_3216Metric" (at 147.32 52.578 90)
+    (property "Footprint" "Resistor_SMD:R_0603_1608Metric" (at 147.32 52.578 90)
       (effects (font (size 1.27 1.27)) hide)
     )
