File: KiCadFiles/FaultSignalGenerator/FaultSignalGenerator_Isaiah_16Channel.kicad_pcb (KiCad board)
At the start: 4 copper layers, 126.2 x 113.3 mm, 280 parts, among them J1 Conn_02x20_Odd_Even, J2 Conn_02x16_Odd_Even, J3 DB25_Receptacle, U1 MCP4431-503E/ST, U10 TL074CDR, U11 TL074CDR, U12 TL074CDR, U13 TL074CDR, U14 PCM1681PWP, U15 PCM1681PWP, U16 TL780-05CKTTR, U2 MCP4431-503E/ST, U3 MCP4431-503E/ST, U4 MCP4431-503E/ST, U5 TL074CDR, U6 TL074CDR, U7 TL074CDR, U8 TL074CDR, U9 TL074CDR

Commit message: Corrected 90+ degree power trace angles
Routing:
- net +6V: track 248.9 -> 242.4 mm
- net +5V: track 408.8 -> 405.8 mm
- net +12V: track 251.1 -> 249.5 mm
